File: glucometer-pcb.kicad_sch (KiCad schematic)
At the start: 19 parts, among them IC3 RC4558IP

Commit message: asd
Parts:
- added BZ1: Buzzer, Buzzer_Beeper:MagneticBuzzer_Kingstate_KCG0601, symbol Device:Buzzer
- added D3: LED, LED_THT:LED_D3.0mm_FlatTop, symbol Device:LED
- added R9: 120, Resistor_THT:R_Axial_DIN0414_L11.9mm_D4.5mm_P15.24mm_Horizontal, symbol Device:R
- added U1: ESP32_DevKit_V1_DOIT, esp32_devkit_v1_doit:esp32_devkit_v1_doit, symbol esp32_devkit_v1_doit:ESP32_DevKit_V1_DOIT
- C1: value (none) -> 10u; footprint (none) -> Capacitor_THT:CP_Radial_Tantal_D7.0mm_P5.00mm
- C2: value (none) -> 15p; footprint (none) -> Capacitor_THT:CP_Radial_D8.0mm_P3.80mm
- C3: value (none) -> 100n; footprint (none) -> Capacitor_THT:CP_Radial_Tantal_D7.0mm_P5.00mm
- D1: value (none) -> LED; footprint (none) -> LED_THT:LED_D3.0mm_Clear
- D2: value (none) -> D_Photo; footprint (none) -> LED_SMD:LED_2010_5025Metric
- IC1: value (none) -> RC4558IP; footprint (none) -> Custom:DIP794W53P254L959H508Q8N
- IC2: value (none) -> LM1458N; footprint (none) -> Custom:MC1458N
- IC3: footprint (none) -> Custom:DIP794W53P254L959H508Q8N
- R1, R2: value (none) -> 10k
- R3: value (none) -> 240; footprint (none) -> Resistor_THT:R_Axial_DIN0414_L11.9mm_D4.5mm_P15.24mm_Horizontal
- R4, R8: value (none) -> 100k; footprint (none) -> Resistor_THT:R_Axial_DIN0414_L11.9mm_D4.5mm_P15.24mm_Horizontal
- R5: value (none) -> 25k; footprint (none) -> Resistor_THT:R_Axial_DIN0414_L11.9mm_D4.5mm_P15.24mm_Horizontal
- R6: value (none) -> 330k; footprint (none) -> Resistor_THT:R_Axial_DIN0414_L11.9mm_D4.5mm_P15.24mm_Horizontal
- R7: value (none) -> 1k; footprint (none) -> Resistor_THT:R_Axial_DIN0414_L11.9mm_D4.5mm_P15.24mm_Horizontal
- TP1, TP2: footprint (none) -> TestPoint:TestPoint_Keystone_5015_Micro-Minature
- TP3: value (none) -> TestPoint; footprint (none) -> TestPoint:TestPoint_Keystone_5015_Micro-Minature
Connections:
- net GND: no longer R3.2
- net VCC: now also BZ1.2 (+), U1.1 (3V3)
- new net: D3.1 (K), R3.2, U1.17 (GND)
- new net: D3.2 (A), U1.23 (D25)
- new net: BZ1.1 (-), R9.1
- new net: R9.2, U1.2 (GND)
Other:
- moved on the sheet: C2, C3, D1, D2, IC2, R3, R4, R6

Commit message: pcb backup
Parts:
- removed TP3: TestPoint, TestPoint:TestPoint_Keystone_5015_Micro-Minature, symbol Connector:TestPoint
- R1, R2, R5: footprint Resistor_THT:R_Axial_DIN0414_L11.9mm_D4.5mm_P15.24mm_Horizontal -> Resistor_THT:R_Axial_DIN0204_L3.6mm_D1.6mm_P7.62mm_Horizontal
- R3: renamed from R9; footprint Resistor_THT:R_Axial_DIN0414_L11.9mm_D4.5mm_P15.24mm_Horizontal -> Resistor_THT:R_Axial_DIN0204_L3.6mm_D1.6mm_P7.62mm_Horizontal
- R4: renamed from R3; footprint Resistor_THT:R_Axial_DIN0414_L11.9mm_D4.5mm_P15.24mm_Horizontal -> Resistor_THT:R_Axial_DIN0204_L3.6mm_D1.6mm_P7.62mm_Horizontal
- R6: renamed from R4; footprint Resistor_THT:R_Axial_DIN0414_L11.9mm_D4.5mm_P15.24mm_Horizontal -> Resistor_THT:R_Axial_DIN0204_L3.6mm_D1.6mm_P7.62mm_Horizontal
- R7: renamed from R6; footprint Resistor_THT:R_Axial_DIN0414_L11.9mm_D4.5mm_P15.24mm_Horizontal -> Resistor_THT:R_Axial_DIN0204_L3.6mm_D1.6mm_P7.62mm_Horizontal
- R8: renamed from R7; footprint Resistor_THT:R_Axial_DIN0414_L11.9mm_D4.5mm_P15.24mm_Horizontal -> Resistor_THT:R_Axial_DIN0204_L3.6mm_D1.6mm_P7.62mm_Horizontal
- R9: renamed from R8; footprint Resistor_THT:R_Axial_DIN0414_L11.9mm_D4.5mm_P15.24mm_Horizontal -> Resistor_THT:R_Axial_DIN0204_L3.6mm_D1.6mm_P7.62mm_Horizontal
- renumbered D3 to D2, D2 to D3
Connections:
- net VCC: no longer BZ1.2 (+)
- net SIGNAL_OUT: now reaches IC3.6 (2IN-), R8.1, R9.2
- net SIGNAL_OUT: now also U1.8 (D5)
- net at R3.1: now also BZ1.2 (+); no longer BZ1.1 (-)
- net at U1.4 (D2): now also BZ1.1 (-)
Other:
- moved on the sheet: BZ1, R3
