File: glucometer-pcb.kicad_pcb (KiCad board)
At the start: 2 copper layers, 17 parts, among them IC1 RC4558IP, IC2 LM1458N, IC3 RC4558IP

Commit message: asd
Parts:
- added BZ1: Buzzer, Buzzer_Beeper:MagneticBuzzer_Kingstate_KCG0601, F.Cu at (139.7, 83.8)
- added D1: LED, LED_THT:LED_D3.0mm_Clear, F.Cu at (94.0, 91.4)
- added D3: LED, LED_THT:LED_D3.0mm_FlatTop, F.Cu at (94.0, 59.0)
- added R3: 240, Resistor_THT:R_Axial_DIN0414_L11.9mm_D4.5mm_P15.24mm_Horizontal, F.Cu at (94.0, 81.9)
- added R9: 120, Resistor_THT:R_Axial_DIN0414_L11.9mm_D4.5mm_P15.24mm_Horizontal, F.Cu at (139.7, 76.2)
- added U1: ESP32_DevKit_V1_DOIT, esp32_devkit_v1_doit:esp32_devkit_v1_doit, F.Cu at (119.4, 83.8)
- moved D2 137.2 mm to (116.8, 162.6), turned to 0 degrees
- moved TP3 100.2 mm to (94.0, 142.2), turned to 180 degrees
- moved C1 98.3 mm to (139.7, 144.2), turned to 90 degrees
- moved C2 91.2 mm to (129.5, 144.2), turned to 90 degrees
- moved IC2 89.6 mm to (110.5, 143.5), turned to 180 degrees
- moved C3 88.3 mm to (119.4, 144.2), turned to 90 degrees
- moved TP1 83.3 mm to (94.0, 132.1), turned to 180 degrees
- moved R8 76.3 mm to (139.7, 131.5), turned to 90 degrees
- moved TP2 68.3 mm to (94.0, 121.9), turned to 180 degrees
- moved R4 62.9 mm to (119.4, 131.5), turned to 90 degrees
- moved IC3 56.8 mm to (106.7, 124.5), turned to 180 degrees
- moved R1 48.6 mm to (139.7, 111.2), turned to 90 degrees
- moved IC1 43.7 mm to (96.5, 103.5), turned to 180 degrees
- moved R6 39.7 mm to (129.5, 116.2), turned to -90 degrees
- moved R7 24.3 mm to (129.5, 95.9), turned to -90 degrees
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
Commit message: pcb backup
Parts:
- removed the D3 at (94.0, 59.0)
- removed the R6 at (129.5, 116.2)
- removed TP3: TestPoint, TestPoint:TestPoint_Keystone_5015_Micro-Minature
- added D2: LED, LED_THT:LED_D3.0mm_FlatTop, F.Cu at (170.0, 97.3)
- added R4: 240, Resistor_THT:R_Axial_DIN0204_L3.6mm_D1.6mm_P7.62mm_Horizontal, F.Cu at (166.0, 89.6)
- R1, R2, R5: footprint Resistor_THT:R_Axial_DIN0414_L11.9mm_D4.5mm_P15.24mm_Horizontal -> Resistor_THT:R_Axial_DIN0204_L3.6mm_D1.6mm_P7.62mm_Horizontal
- R3: value 240 -> 120; footprint Resistor_THT:R_Axial_DIN0414_L11.9mm_D4.5mm_P15.24mm_Horizontal -> Resistor_THT:R_Axial_DIN0204_L3.6mm_D1.6mm_P7.62mm_Horizontal
- R6: renamed from R4; footprint Resistor_THT:R_Axial_DIN0414_L11.9mm_D4.5mm_P15.24mm_Horizontal -> Resistor_THT:R_Axial_DIN0204_L3.6mm_D1.6mm_P7.62mm_Horizontal
- R7: value 1k -> 330k; footprint Resistor_THT:R_Axial_DIN0414_L11.9mm_D4.5mm_P15.24mm_Horizontal -> Resistor_THT:R_Axial_DIN0204_L3.6mm_D1.6mm_P7.62mm_Horizontal
- R8: value 100k -> 1k; footprint Resistor_THT:R_Axial_DIN0414_L11.9mm_D4.5mm_P15.24mm_Horizontal -> Resistor_THT:R_Axial_DIN0204_L3.6mm_D1.6mm_P7.62mm_Horizontal
- R9: value 120 -> 100k; footprint Resistor_THT:R_Axial_DIN0414_L11.9mm_D4.5mm_P15.24mm_Horizontal -> Resistor_THT:R_Axial_DIN0204_L3.6mm_D1.6mm_P7.62mm_Horizontal
- U1: footprint esp32_devkit_v1_doit:esp32_devkit_v1_doit -> esp32_devkit_v1_doit:esp32_devkit_v1_doit_own_ESP
- moved R3 114.5 mm to (204.5, 111.8), turned to 0 degrees
- moved R9 93.0 mm to (199.8, 147.2), turned to 180 degrees
- moved R2 92.3 mm to (198.7, 118.4), turned to 180 degrees
- moved R7 90.7 mm to (198.7, 154.7), turned to 180 degrees
- moved R5 87.9 mm to (193.1, 143.8), turned to 0 degrees
- moved IC1 86.9 mm to (182.7, 114.5), turned to -90 degrees
- moved BZ1 77.9 mm to (208.4, 120.5), turned to 180 degrees
- moved IC3 76.6 mm to (182.9, 132.1), turned to 0 degrees
- moved D1 76.2 mm to (169.1, 103.8), turned to 180 degrees
- moved TP1 74.3 mm to (166.8, 117.7), turned to 0 degrees
- moved TP2 73.0 mm to (166.8, 127.0), turned to 0 degrees
- moved U1 72.4 mm to (190.4, 97.8)
- moved D3 70.4 mm to (186.9, 170.2), turned to 180 degrees
- moved IC2 69.0 mm to (179.2, 149.9), turned to 90 degrees
- moved C3 67.0 mm to (183.1, 123.4), turned to 180 degrees
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- renumbered D2 to D3
Connections:
- BZ1 pad 2: VCC -> Net-(BZ1-Pad2)
- IC3 pad 6: Net-(IC3-Pad6) -> SIGNAL_OUT
- R3 pad 1: Net-(D1-Pad2) -> Net-(BZ1-Pad2)
- R3 pad 2: Net-(D3-Pad1) -> Net-(R3-Pad2)
- R7 pad 1: Net-(IC3-Pad6) -> /SIGNAL_1
- R7 pad 2: /PWD_1.65 -> Net-(C2-Pad2)
- R8 pad 1: Net-(IC3-Pad7) -> SIGNAL_OUT
- R8 pad 2: Net-(IC3-Pad6) -> /PWD_1.65
- R9 pad 1: Net-(BZ1-Pad1) -> Net-(IC3-Pad7)
- R9 pad 2: Net-(R9-Pad2) -> SIGNAL_OUT
- U1 pad 17: Net-(D3-Pad1) -> Net-(D2-Pad1)
- U1 pad 2: Net-(R9-Pad2) -> Net-(R3-Pad2)
- U1 pad 4: unconnected-(U1-Pad4) -> Net-(BZ1-Pad1)
- U1 pad 8: unconnected-(U1-Pad8) -> SIGNAL_OUT
Routing:
- net VCC: track 0.00 -> 298.1 mm
- net GND: track 0.00 -> 108.0 mm
- net /PWD_1.65: track 0.00 -> 93.5 mm
- net Net-(BZ1-Pad1): track 0.00 -> 52.8 mm
- net Net-(C2-Pad2): track 0.00 -> 52.3 mm
- net Net-(R3-Pad2): track 0.00 -> 50.7 mm
- net /SIGNAL_1: track 0.00 -> 47.7 mm
- net Net-(IC1-Pad3): track 0.00 -> 37.6 mm
- net Net-(D2-Pad1): track 0.00 -> 35.7 mm
- net SIGNAL_OUT: track 0.00 -> 26.7 mm
- net Net-(IC3-Pad7): track 0.00 -> 22.7 mm
- net Net-(C2-Pad1): track 0.00 -> 22.1 mm
- net Net-(D2-Pad2): track 0.00 -> 19.4 mm
- net Net-(C1-Pad1): track 0.00 -> 19.4 mm
- net Net-(D1-Pad2): track 0.00 -> 14.5 mm
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
Commit message: prototype PCB
Parts:
- moved TP2 6.89 mm to (172.0, 122.4)
- moved R8 5.65 mm to (198.6, 156.7)
- moved R9 5.33 mm to (201.0, 152.4)
- moved R5 5.26 mm to (193.9, 149.0)
- moved R7 5.21 mm to (198.7, 159.9)
- moved TP1 5.19 mm to (172.0, 117.6)
- moved D3 5.04 mm to (186.9, 175.2)
- moved IC2 5.04 mm to (179.2, 154.9)
- moved R6 5.04 mm to (177.8, 167.1)
- moved C2 5.04 mm to (182.6, 160.8)
- moved D1 3.36 mm to (172.3, 105.1)
- moved IC3 2.86 mm to (181.3, 134.5)
- moved C1 2.61 mm to (190.4, 133.4)
- moved BZ1 2.55 mm to (205.9, 121.3)
- moved R3 2.11 mm to (202.4, 111.9)
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Routing:
- net VCC: track 298.1 -> 183.1 mm
- net SIGNAL_OUT: track 26.7 -> 113.5 mm
- net Net-(IC3-Pad7): track 22.7 -> 50.0 mm
- net /SIGNAL_1: track 47.7 -> 60.0 mm
- net /PWD_1.65: track 93.5 -> 87.0 mm
- net /SIGNAL_2: track 13.1 -> 17.5 mm
- net Net-(D1-Pad2): track 14.5 -> 17.0 mm
- net Net-(C2-Pad2): track 52.3 -> 50.4 mm
- net Net-(BZ1-Pad2): track 10.6 -> 9.59 mm
- net Net-(C1-Pad1): track 19.4 -> 20.2 mm
- net Net-(R3-Pad2): track 50.7 -> 50.0 mm

Commit message: last update pcb
Parts:
- moved R3 36.3 mm to (166.6, 118.1)
- moved BZ1 35.9 mm to (172.0, 109.8)
- moved D1 34.9 mm to (173.1, 140.0)
- moved D2 33.5 mm to (170.1, 130.8)
- moved TP2 33.1 mm to (171.7, 155.5)
- moved R4 32.6 mm to (166.6, 122.2)
- moved IC1 31.4 mm to (201.8, 139.4)
- moved TP1 31.4 mm to (171.7, 149.0)
- moved U1 16.5 mm to (193.0, 114.1)
- moved R2 14.2 mm to (204.8, 130.9)
- moved R1 14.1 mm to (204.7, 127.1)
- moved C3 9.14 mm to (190.5, 128.7), turned to 90 degrees
Routing:
- net Net-(R3-Pad2): track 50.0 -> 77.4 mm
- net Net-(BZ1-Pad1): track 52.6 -> 79.1 mm
- net Net-(IC1-Pad3): track 37.6 -> 15.6 mm
- net Net-(D2-Pad1): track 35.7 -> 54.9 mm
- net Net-(D2-Pad2): track 19.4 -> 37.6 mm
- net /PWD_1.65: track 87.0 -> 102.6 mm
- net /SIGNAL_1: track 60.0 -> 71.2 mm
- net SIGNAL_OUT: track 113.5 -> 104.7 mm
- net VCC: track 183.1 -> 176.5 mm
- net GND: track 107.6 -> 112.7 mm
- net Net-(C1-Pad1): track 20.2 -> 23.0 mm
- net Net-(D1-Pad2): track 17.0 -> 19.1 mm
